File: bluepillcarrier/bluepillcarrier.kicad_sch (KiCad schematic)
At the start: 70 parts, among them CN1 USB, CN2 Can, CN3 Can, CN4 RTC, CN5 RS485, CN6 485, CN7 BME, CN8 SWD, Q1 SS8050, SW1 Usr1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

Commit message: Some updates and fixes
Parts:
- added JP3: USB pwr, Connector_PinHeader_2.54mm:PinHeader_1x02_P2.54mm_Vertical, symbol Jumper:Jumper_2_Open
Connections:
- net 3V3: no longer C3.1
- net 5V: now also C3.1, JP3.2 (B); no longer D1.1 (K)
- new net: D1.1 (K), JP3.1 (A)
Other:
- note added: "RTC Slave Address: 0x68 BME Slave Address: 0x77"
- note added: "Slave Address: 0x60"
Changed lines of the file:
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@@
 		)
 	)
+	(text "RTC Slave Address: 0x68\nBME Slave Address: 0x77"
+		(exclude_from_sim no)
+		(at 345.694 189.992 0)
+		(effects
+			(font
+				(size 2.54 2.54)
+			)
+		)
+	)
 	(text "Alternative JLCPCB part: C709357\nOriginal: C165948"
 		(exclude_from_sim no)
@@
 		)
 	)
+	(text "Slave Address: 0x60"
+		(exclude_from_sim no)
+		(at 187.452 142.24 0)
+		(effects
+			(font
+				(size 2.54 2.54)
+			)
+		)
+	)
 	(text_box "WKUP"
 		(exclude_from_sim no)
@@
 	(wire
 		(pts
+			(xy 69.85 213.36) (xy 71.12 213.36)
+		)
+		(stroke
+			(width 0)
+			(type default)
+		)
+	)
+	(wire
+		(pts
 			(xy 327.66 173.99) (xy 332.74 173.99)
 		)
@@
 		)
 	)
+	(label "5V"
+		(at 132.08 158.75 90)
+		(effects
+			(font
+				(size 1.27 1.27)
+			)
+			(justify left bottom)
+		)
+	)
 	(label "TX3"
 		(at 335.28 109.22 0)
@@
 		)
 	)
-	(label "3V3"
-		(at 132.08 158.75 90)
-		(effects
-			(font
-				(size 1.27 1.27)
-			)
-			(justify left bottom)
-		)
-	)
 	(label "RO"
 		(at 274.32 45.72 180)
@@
 	)
 	(label "5V"
-		(at 81.28 213.36 180)
+		(at 69.85 213.36 180)
 		(effects
 			(font
@@
 					(unit 1)
 				)
+			)
+		)
+	)
+	(symbol
+		(lib_id "Jumper:Jumper_2_Open")
+		(at 76.2 213.36 180)
+		(unit 1)
+		(exclude_from_sim no)
+		(in_bom yes)
+		(on_board yes)
+		(dnp no)
+		(fields_autoplaced yes)
+		(property "Reference" "JP3"
+			(at 76.2 208.28 0)
+			(effects
+				(font
+					(size 1.27 1.27)
+				)
+			)
+		)
+		(property "Value" "USB pwr"
+			(at 76.2 210.82 0)
+			(effects
+				(font
+					(size 1.27 1.27)
+				)
+			)
+		)
+		(property "Footprint" "Connector_PinHeader_2.54mm:PinHeader_1x02_P2.54mm_Vertical"
+			(at 76.2 213.36 0)
+			(effects
+				(font
+					(size 1.27 1.27)
+				)
+				(hide yes)
+			)
+		)
+		(property "Datasheet" "~"
+			(at 76.2 213.36 0)
+			(effects
+				(font
+					(size 1.27 1.27)
+				)
+				(hide yes)
+			)
+		)
+		(property "Description" "Jumper, 2-pole, open"
+			(at 76.2 213.36 0)
+			(effects
+				(font
+					(size 1.27 1.27)
+				)
+				(hide yes)
+			)
+		)
+		(property "Note" ""
+			(at 76.2 213.36 0)
+			(effects
+				(font
+					(size 1.27 1.27)
+				)
+				(hide yes)
+			)
+		)
+		(property "LCSC" "C5360898"
+			(at 76.2 213.36 90)
+			(effects
+				(font
+					(size 1.27 1.27)
+				)
+				(hide yes)
+			)
+		)
+		(pin "1"
+		)
+		(pin "2"
+		)
+		(instances
+			(project "bluepillcarrier"
+				(path "/a1c59454-a06f-4e3a-accb-f295f4aa94b3"
+					(reference "JP3")
+					(unit 1)
+				)

Commit message: Fixes: - Corrected OLED footprint - Green led resistor set to 1k - Updated all the labels to 1mm for better visibility - Moved trimmer a bit below to save a bit of space for buttons
Parts:
- JP1: value RS485 Term -> CAN Term
- R10, R11, R2, R21, R23, R27, R28, R4, R6, R9: value 330 -> 1k; LCSC C25104 -> C140196
Changed lines of the file:
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@@
 			)
 		)
-		(property "Value" "330"
+		(property "Value" "1k"
 			(at 60.325 128.2699 0)
 			(effects
@@
 			)
 		)
-		(property "LCSC" "C25104"
+		(property "LCSC" "C140196"
 			(at 58.42 127 0)
 			(effects
@@
 			)
 		)
-		(property "Value" "330"
+		(property "Value" "1k"
 			(at 108.585 128.2699 0)
 			(effects
@@
 			)
 		)
-		(property "LCSC" "C25104"
+		(property "LCSC" "C140196"
 			(at 106.68 127 0)
 			(effects
@@
 			)
 		)
-		(property "Value" "330"
+		(property "Value" "1k"
 			(at 93.345 128.2699 0)
 			(effects
@@
 			)
 		)
-		(property "LCSC" "C25104"
+		(property "LCSC" "C140196"
 			(at 91.44 127 0)
 			(effects
@@
 			)
 		)
-		(property "Value" "330"
+		(property "Value" "1k"
 			(at 295.275 129.5399 0)
 			(effects
@@
 			)
 		)
-		(property "LCSC" "C25104"
+		(property "LCSC" "C140196"
 			(at 293.37 128.27 0)
 			(effects
@@
 			)
 		)
-		(property "Value" "RS485 Term"
+		(property "Value" "CAN Term"
 			(at 180.34 187.9599 90)
 			(effects
@@
 			)
 		)
-		(property "Value" "330"
+		(property "Value" "1k"
 			(at 76.835 128.2699 0)
 			(effects
@@
 			)
 		)
-		(property "LCSC" "C25104"
+		(property "LCSC" "C140196"
 			(at 74.93 127 0)
 			(effects
@@
 			)
 		)
-		(property "Value" "330"
+		(property "Value" "1k"
 			(at 315.595 129.5399 0)
 			(effects
@@
 			)
 		)
-		(property "LCSC" "C25104"
+		(property "LCSC" "C140196"
 			(at 313.69 128.27 0)
 			(effects
@@
 			)
 		)
-		(property "Value" "330"
+		(property "Value" "1k"
 			(at 43.815 128.2699 0)
 			(effects
@@
 			)
 		)
-		(property "LCSC" "C25104"
+		(property "LCSC" "C140196"
 			(at 41.91 127 0)
 			(effects
@@
 			)
 		)
-		(property "Value" "330"
+		(property "Value" "1k"
 			(at 125.095 128.2699 0)
 			(effects
@@
 			)
 		)
-		(property "LCSC" "C25104"
+		(property "LCSC" "C140196"
 			(at 123.19 127 0)
 			(effects
@@
 			)
 		)
-		(property "Value" "330"
+		(property "Value" "1k"
 			(at 337.185 129.5399 0)
 			(effects
@@
 			)
 		)
-		(property "LCSC" "C25104"
+		(property "LCSC" "C140196"
 			(at 335.28 128.27 0)
 			(effects
@@
 			)
 		)
-		(property "Value" "330"
+		(property "Value" "1k"
 			(at 273.685 129.5399 0)
 			(effects
@@
 			)
 		)
-		(property "LCSC" "C25104"
+		(property "LCSC" "C140196"
 			(at 271.78 128.27 0)
 			(effects

Commit message: Some additional fixes
Parts:
- removed U4: 25LCxxx, Package_SO:SO-8_3.9x4.9mm_P1.27mm, symbol Memory_EEPROM:25LCxxx
- added U2: M95512-WMN6TP, Package_SO:SOIC-8_3.9x4.9mm_P1.27mm, symbol Memory_EEPROM:M95256-WMN6P
- OLED1: footprint oled:MODULE_DM-OLED096-636 -> bluepill:MODULE_DM-OLED096-636
Connections:
- net 3V3: now also U2.8 (VCC)
- net CS: now also U2.1 (~{S})
- net DI: now also LD12.2 (A), MODULE1.35 (PB10); no longer LD10.2 (A), MODULE1.6 (PA9)
- net GND: now also U2.4 (VSS)
- net MISO: now also U2.2 (Q)
- net MOSI: now also U2.5 (D)
- net RO: now also LD11.2 (A), MODULE1.36 (PB11); no longer LD9.2 (A), MODULE1.7 (PA10)
- net SCK: now also U2.6 (C)
- net at R13.2: now also U2.3 (~{W})
- net at R12.2: now also U2.7 (~{HOLD})
- removed net RX3: LD11.2 (A), MODULE1.36 (PB11), U1.6 (TXD)
- removed net TX3: LD12.2 (A), MODULE1.35 (PB10), U1.7 (RXD)
- new net RX1: LD9.2 (A), MODULE1.7 (PA10), U1.6 (TXD)
- new net TX1: LD10.2 (A), MODULE1.6 (PA9), U1.7 (RXD)
Changed lines of the file:
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@@
 		)
 	)
-	(label "RX1"
+	(label "RX3"
 		(at 373.38 80.01 180)
 		(effects
@@
 		)
 	)
-	(label "RX3"
+	(label "RX1"
 		(at 29.21 219.71 180)
 		(effects
@@
 		)
 	)
-	(label "TX3"
+	(label "TX1"
 		(at 29.21 222.25 180)
 		(effects
@@
 		)
 	)
-	(label "TX1"
+	(label "TX3"
 		(at 373.38 86.36 180)
 		(effects
@@
 	)
 	(symbol
-		(lib_id "Memory_EEPROM:25LCxxx")
-		(at 177.8 229.87 0)
-		(unit 1)
-		(exclude_from_sim no)
-		(in_bom yes)
-		(on_board yes)
-		(dnp no)
-		(fields_autoplaced yes)
-		(property "Reference" "U4"
-			(at 179.9433 219.71 0)
-			(effects
-				(font
-					(size 1.27 1.27)
-				)
-				(justify left)
-			)
-		)
-		(property "Value" "25LCxxx"
-			(at 179.9433 222.25 0)
-			(effects
-				(font
-					(size 1.27 1.27)
-				)
-				(justify left)
-			)
-		)
-		(property "Footprint" "Package_SO:SO-8_3.9x4.9mm_P1.27mm"
-			(at 177.8 229.87 0)
-			(effects
-				(font
-					(size 1.27 1.27)
-				)
-				(hide yes)
-			)
-		)
-		(property "Datasheet" "http://ww1.microchip.com/downloads/en/DeviceDoc/21832H.pdf"
-			(at 177.8 229.87 0)
-			(effects
-				(font
-					(size 1.27 1.27)
-				)
-				(hide yes)
-			)
-		)
-		(property "Description" "SPI Serial EEPROM, DIP-8/SOIC-8/TSSOP-8"
-			(at 177.8 229.87 0)
-			(effects
-				(font
-					(size 1.27 1.27)
-				)
-				(hide yes)
-			)
-		)
-		(property "LCSC" "C84670"
-			(at 177.8 229.87 0)
-			(effects
-				(font
-					(size 1.27 1.27)
-				)
-				(hide yes)
-			)
-		)
-		(pin "4"
-		)
-		(pin "8"
-		)
-		(pin "7"
-		)
-		(pin "3"
-		)
-		(pin "5"
-		)
-		(pin "6"
-		)
-		(pin "1"
-		)
-		(pin "2"
-		)
-		(instances
-			(project "bluepillcarrier"
-				(path "/a1c59454-a06f-4e3a-accb-f295f4aa94b3"
-					(reference "U4")
-					(unit 1)
-				)
-			)
-		)
-	)
-	(symbol
 		(lib_id "Device:C")
 		(at 200.66 209.55 0)
@@
 			)
 		)
-		(property "Footprint" "oled:MODULE_DM-OLED096-636"
+		(property "Footprint" "bluepill:MODULE_DM-OLED096-636"
 			(at 200.66 121.92 0)
 			(effects
@@
 					(unit 1)
 				)
+			)
+		)
+	)
+	(symbol
+		(lib_id "Memory_EEPROM:M95256-WMN6P")
+		(at 177.8 229.87 0)
+		(unit 1)
+		(exclude_from_sim no)
+		(in_bom yes)
+		(on_board yes)
+		(dnp no)
+		(fields_autoplaced yes)
+		(property "Reference" "U2"
+			(at 179.9433 219.71 0)
+			(effects
+				(font
+					(size 1.27 1.27)
+				)
+				(justify left)
+			)
+		)
+		(property "Value" "M95512-WMN6TP"
+			(at 179.9433 222.25 0)
+			(effects
+				(font
+					(size 1.27 1.27)
+				)
+				(justify left)
+			)
+		)
+		(property "Footprint" "Package_SO:SOIC-8_3.9x4.9mm_P1.27mm"
+			(at 177.8 229.87 0)
+			(effects
+				(font
+					(size 1.27 1.27)
+				)
+				(hide yes)
+			)
+		)
+		(property "Datasheet" "http://www.st.com/content/ccc/resource/technical/document/datasheet/9d/75/f0/3e/76/00/4c/0b/CD00103810.pdf/files/CD00103810.pdf/jcr:content/translations/en.CD00103810.pdf"
+			(at 177.8 229.87 0)
+			(effects
+				(font
+					(size 1.27 1.27)
+				)
+				(hide yes)
+			)
+		)
+		(property "Description" "SPI EEPROM, 512Kb (32K x 8), No Identification Page, 2.5 to 5.5V, SO8"
+			(at 177.8 229.87 0)
+			(effects
+				(font
+					(size 1.27 1.27)
+				)
+				(hide yes)
+			)
+		)
+		(property "LCSC" "C7567"
+			(at 177.8 229.87 0)
+			(effects
+				(font
+					(size 1.27 1.27)
+				)
+				(hide yes)
+			)
+		)
+		(pin "8"
+		)
+		(pin "5"
+		)
+		(pin "3"
+		)
+		(pin "4"
+		)
+		(pin "7"
+		)
+		(pin "2"
+		)
+		(pin "1"
+		)
+		(pin "6"
+		)
+		(instances
+			(project "bluepillcarrier"
+				(path "/a1c59454-a06f-4e3a-accb-f295f4aa94b3"
+					(reference "U2")
+					(unit 1)
+				)

Commit message: minor
Parts:
- U3: LCSC (none) -> C38695
Changed lines of the file:
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@@
+			)
+		)
+		(property "LCSC" "C38695"
+			(at 163.83 163.83 0)
+			(effects
+				(font
+					(size 1.27 1.27)
+				)
+				(hide yes)
 			)
 		)

Commit message: some updates
Parts:
- LD10, LD11, LD12, LD9: LCSC C12624 -> C2288
Connections:
- net 3V3: now also LD10.2 (A), LD11.2 (A), LD12.2 (A), LD9.2 (A)
- net DI: now also R28.2; no longer LD12.2 (A)
- net GND: no longer R21.2, R23.2, R27.2, R28.2
- net RO: now also R27.2; no longer LD11.2 (A)
- net RX1: now also R21.2; no longer LD9.2 (A)
- net TX1: now also R23.2; no longer LD10.2 (A)

Commit message: - changed temperature sensor
Parts:
- removed U5: LM35-D, Package_SO:SOIC-8_3.9x4.9mm_P1.27mm, symbol Sensor_Temperature:LM35-D
- added U4: TMP102xxDRL, Package_TO_SOT_SMD:SOT-563, symbol Sensor_Temperature:TMP102xxDRL
Connections:
- net 3V3: now also C5.1, U4.5 (V+)
- net 5V: no longer C5.1
- net GND: now also U4.2 (GND), U4.4 (ADD0)
- net PA2: now also U4.3 (ALERT)
- net SCL1: now also U4.1 (SCL)
- net SDA1: now also U4.6 (SDA)
Other:
- note added: "Slave Address: 0x48"

Commit message: Some updates
Parts:
- added CN9: Lin, Connector_PinHeader_2.54mm:PinHeader_1x03_P2.54mm_Vertical, symbol Connector:Conn_01x03_Pin
- added D2: 1N4148W, Diode_SMD:D_SOD-123, symbol Diode:1N4148W
- added JP4: Lin_Vbat, Connector_PinHeader_2.54mm:PinHeader_1x03_P2.54mm_Vertical, symbol Jumper:Jumper_3_Open
- added JP5: Lin master, Connector_PinHeader_2.54mm:PinHeader_1x02_P2.54mm_Vertical, symbol Jumper:Jumper_2_Open
- added LD13: Rx, LED_SMD:LED_0603_1608Metric, symbol Device:LED
- added LD14: Tx, LED_SMD:LED_0603_1608Metric, symbol Device:LED
- added R29, R30, R31: 1k, Resistor_SMD:R_0402_1005Metric, symbol Device:R
- added U5: TJA1029T, Package_SO:SOIC-8_3.9x4.9mm_P1.27mm, symbol Interface_CAN_LIN:TJA1029T
- CN3, CN6: now not fitted
- CN8: now left out of the parts list
Connections:
- net 3V3: now also LD13.2 (A), LD14.2 (A)
- net 5V: now also JP4.1 (A), U5.2 (~{SLP})
- net GND: now also CN9.1 (Pin_1), U5.5 (GND)
- net PA15: now reaches MODULE1.10 (PA15)
- net PA15: now also R17.1
- net PA2: no longer names the net of U4.3 (ALERT)
- net PA2: no longer MODULE1.27 (PA2)
- net PA3 renamed RX2
- net RX2: now also R30.2, U5.1 (RXD); no longer R17.1
- new net: LD14.1 (K), R31.1
- new net: D2.1 (K), R29.1
- new net: JP4.2 (C), U5.7 (VBAT)
- new net: LD13.1 (K), R30.1
- new net: JP5.1 (A), R29.2
- new net Lin: CN9.2 (Pin_2), JP5.2 (B), U5.6 (LIN)
- new net Lin_Vbat: CN9.3 (Pin_3), D2.2 (A), JP4.3 (B)
- new net TX2: MODULE1.27 (PA2), R31.2, U5.4 (TXD)

Commit message: some minor modifications
Other:
- note added: "Slave Address: 0x3C"
- note removed: "Slave Address: 0x60"
Changed lines of the file:
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@@
 		)
 	)
-	(text "Slave Address: 0x60"
+	(text "Slave Address: 0x3C"
 		(exclude_from_sim no)
 		(at 187.452 142.24 0)
