File: bluepillcarrier/bluepillcarrier.kicad_sch (KiCad schematic)
At the start: 81 parts, among them CN1 USB, CN2 Can, CN3 Can, CN4 RTC, CN5 RS485, CN6 485, CN7 BME, CN8 SWD, CN9 Lin, Q1 SS8050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

Commit message: some updates
Parts:
- removed BZ1: Buzzer, Buzzer_Beeper:Buzzer_12x9.5RM7.6, symbol Device:Buzzer
- removed Q1: SS8050, Package_TO_SOT_SMD:SOT-23, symbol Transistor_BJT:SS8050
- added C6: 100nF, Capacitor_SMD:C_0402_1005Metric, symbol Device:C
- added CN10: IO, Connector_PinSocket_2.54mm:PinSocket_1x07_P2.54mm_Vertical, symbol Connector:Conn_01x07_Pin
- added CN11: QWIIC, Connector_JST:JST_SH_SM04B-SRSS-TB_1x04-1MP_P1.00mm_Horizontal, symbol Connector:Conn_01x04_Socket
- added LD15, LD16: Led Blue, LED_SMD:LED_0603_1608Metric, symbol Device:LED
- added R32: 1k, Resistor_SMD:R_0402_1005Metric, symbol Device:R
- added U7: ATECC608A-SSHDA, Package_SO:SOIC-8_3.9x4.9mm_P1.27mm, symbol Security:ATECC608A-SSHDA
- CN4: LCSC C40877 -> C2832269
- LD1, LD2, LD3, LD4, LD5, LD6: value O1_G -> Led Blue; LCSC C12624 -> C2288
- LD10, LD12, LD14: value Tx -> Led Blue
- LD11, LD13, LD9: value Rx -> Led Blue
- LD7: value 3v3 -> Led Red
- LD8: value 5v -> Led Red
Connections:
- net 3V3: now also C6.1, CN10.5 (Pin_5), CN11.2 (Pin_2), LD15.2 (A), LD16.2 (A), U7.8 (VCC)
- net 5V: now also CN10.6 (Pin_6)
- net CANRX: now also R17.2
- net CANTX: now also R32.2
- net GND: now also C6.2, CN10.7 (Pin_7), CN11.1 (Pin_1), U7.4 (GND)
- net Lin_Vbat: no longer D2.2 (A)
- net PA15: now also CN10.1 (Pin_1); no longer R17.1
- net SCL1: now also CN11.4 (Pin_4), U7.6 (SCL)
- net SDA1: now also CN11.3 (Pin_3), U7.5 (SDA)
- net Lin_Vcc: now reaches JP4.2 (C), U5.7 (VBAT)
- net Lin_Vcc: now also D2.2 (A)
- net at MODULE1.22 (PC13): now also CN10.2 (Pin_2)
- net at MODULE1.23 (PC14): now also CN10.3 (Pin_3)
- net at MODULE1.24 (PC15): now also CN10.4 (Pin_4)
- new net: LD15.1 (K), R17.1
- new net: LD16.1 (K), R32.1
- no-connect marks 13 -> 10
Other:
- moved on the sheet: LD10, LD11, LD12, LD13, LD14, LD7, LD8, LD9, R18, R20, R21, R23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
