File: bluepillcarrier/bluepillcarrier.kicad_pcb (KiCad board)
At the start: 4 copper layers, 81.3 x 86.4 mm, 128 parts, among them CN1 USB, CN2 Can, CN3 Can, CN4 RTC, CN5 RS485, CN6 485, CN7 BME, CN8 SWD, Q1 SS8050, SW1 Usr1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

Commit message: Some updates
Parts:
- removed CN3: Can, Connector_PinHeader_2.54mm:PinHeader_1x04_P2.54mm_Vertical
- removed CN6: 485, Connector_PinHeader_2.54mm:PinHeader_1x04_P2.54mm_Vertical
- removed kibuzzard-69594CE1: G***, kibuzzard-69594CE1
- removed kibuzzard-69594CE6: G***, kibuzzard-69594CE6
- removed kibuzzard-69594DCB: G***, kibuzzard-69594DCB
- removed kibuzzard-69594DFC: G***, kibuzzard-69594DFC
- removed kibuzzard-69594E11: G***, kibuzzard-69594E11
- removed kibuzzard-695AB3BA: G***, kibuzzard-695AB3BA
- added CN9: Lin, Connector_PinHeader_2.54mm:PinHeader_1x03_P2.54mm_Vertical, F.Cu at (158.6, 122.6)
- added D2: 1N4148W, Diode_SMD:D_SOD-123, F.Cu at (161.5, 116.2)
- added G***: LOGO, logo:lin, F.Cu at (169.3, 122.2)
- added JP4: Lin_Vbat, Connector_PinHeader_2.54mm:PinHeader_1x03_P2.54mm_Vertical, F.Cu at (171.3, 114.0)
- added JP5: Lin master, Connector_PinHeader_2.54mm:PinHeader_1x02_P2.54mm_Vertical, F.Cu at (166.1, 113.9)
- added LD13: Rx, LED_SMD:LED_0603_1608Metric, F.Cu at (120.4, 80.0)
- added LD14: Tx, LED_SMD:LED_0603_1608Metric, F.Cu at (120.4, 82.8)
- added R29: 1k, Resistor_SMD:R_0402_1005Metric, F.Cu at (161.6, 112.5)
- added R30: 1k, Resistor_SMD:R_0402_1005Metric, F.Cu at (117.1, 80.0)
- added R31: 1k, Resistor_SMD:R_0402_1005Metric, F.Cu at (117.2, 82.8)
- added U5: TJA1029T, Package_SO:SOIC-8_3.9x4.9mm_P1.27mm, F.Cu at (157.2, 115.1)
- added kibuzzard-696A19CC: G***, kibuzzard-696A19CC, F.Cu at (129.1, 104.2)
- added kibuzzard-696A1A13: G***, kibuzzard-696A1A13, F.Cu at (115.5, 113.3)
- added kibuzzard-696A233A: G***, kibuzzard-696A233A, F.Cu at (161.1, 119.8)
- added kibuzzard-696A2374: G***, kibuzzard-696A2374, F.Cu at (168.8, 118.6)
- added kibuzzard-696A237E: G***, kibuzzard-696A237E, F.Cu at (168.9, 114.0)
- added kibuzzard-696A23BE: G***, kibuzzard-696A23BE, F.Cu at (156.4, 110.5)
- added kibuzzard-696A2AD8: G***, kibuzzard-696A2AD8, F.Cu at (166.1, 111.1)
- added kibuzzard-696A4D49: G***, kibuzzard-696A4D49, F.Cu at (123.4, 80.0)
- added kibuzzard-696A4D50: G***, kibuzzard-696A4D50, F.Cu at (123.5, 82.8)
- added kibuzzard-696A4D9E: G***, kibuzzard-696A4D9E, F.Cu at (125.9, 81.4)
- moved R18 59.4 mm to (176.0, 91.1), turned to -90 degrees
- moved R20 56.9 mm to (173.0, 91.1), turned to -90 degrees
- moved LD7 55.8 mm to (176.0, 88.4), turned to 90 degrees
- moved LD8 53.2 mm to (172.9, 88.5), turned to 90 degrees
- moved kibuzzard-69594C8F 52.6 mm to (176.0, 85.4), turned to 90 degrees
- moved kibuzzard-69594C8A 50.1 mm to (172.9, 85.7), turned to 90 degrees
- moved R5 13.2 mm to (185.3, 119.2)
- moved R8 13.2 mm to (185.3, 121.6)
- moved kibuzzard-69594DEB 5.51 mm to (185.1, 87.4)
- moved kibuzzard-69594D1B 5.06 mm to (179.1, 93.5), turned to 0 degrees
- moved Q1 3.04 mm to (119.8, 95.8)
- moved R17 3.01 mm to (123.5, 96.8)
- moved G*** 2.49 mm to (165.1, 94.2)
- moved kibuzzard-69594D45 2.03 mm to (165.1, 77.7)
- moved RV1 1.92 mm to (165.1, 81.3)
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Connections:
- MODULE1 pad 10: unconnected-(MODULE1-PA15-Pad10) -> /PA15
- MODULE1 pad 27: /PA2 -> /TX2
- MODULE1 pad 28: /PA3 -> /RX2
- R17 pad 1: /PA3 -> /PA15
- U4 pad 3: /PA2 -> unconnected-(U4-ALERT-Pad3)
Routing:
- net /RX2: track 0.00 -> 83.0 mm, vias 0 -> 3
- net /TX2: track 0.00 -> 75.3 mm, vias 0 -> 3
- net /PA15: track 0.00 -> 43.6 mm, vias 0 -> 2
- net /PA2: track 39.6 -> 0.00 mm
- net /PA3: track 39.3 -> 0.00 mm
- net /5V: track 145.3 -> 120.7 mm, vias 4 -> 6
- net /A: track 59.0 -> 37.8 mm
- net /B: track 63.5 -> 44.2 mm
- net /Lin: track 0.00 -> 16.8 mm, vias 0 -> 1
- net Net-(JP4-C): track 0.00 -> 15.9 mm, vias 0 -> 1
- net /Lin_Vbat: track 0.00 -> 14.8 mm
- net /CANH: track 58.2 -> 45.9 mm, vias 4 -> 3
- net /CANL: track 55.3 -> 45.1 mm
- net Net-(JP5-A): track 0.00 -> 5.58 mm
- net Net-(CN1-CC1): track 7.20 -> 10.8 mm
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
Commit message: some minor modifications
Parts:
- moved R17 1.62 mm to (123.0, 95.3)
- moved Q1 1.50 mm to (119.6, 94.4)
Routing:
- net Net-(BZ1--): track 8.61 -> 9.99 mm
- net /PA15: track 43.6 -> 42.3 mm
- net GND: vias 182 -> 181
Changed lines of the file:
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@@
 	(footprint "Package_TO_SOT_SMD:SOT-23"
 		(layer "F.Cu")
-		(at 119.81 95.84 180)
+		(at 119.56 94.36 180)
 		(descr "SOT, 3 Pin (JEDEC TO-236 Var AB https://www.jedec.org/document_search?search_api_views_fulltext=TO-236), generated with kicad-footprint-generator ipc_gullwing_generator.py")
 		(tags "SOT TO_SOT_SMD")
@@
 				(font
 					(size 0.001 0.001)
+					(thickness 0.15)
 				)
 			)
@@
 				(font
 					(size 0.001 0.001)
+					(thickness 0.15)
 				)
 			)
@@
 				(font
 					(size 0.001 0.001)
+					(thickness 0.15)
 				)
 			)
@@
 				(font
 					(size 0.001 0.001)
+					(thickness 0.15)
 				)
 			)
@@
 				(font
 					(size 0.001 0.001)
+					(thickness 0.15)
 				)
 			)
@@
 				(font
 					(size 0.001 0.001)
+					(thickness 0.15)
 				)
 			)
@@
 				(font
 					(size 0.001 0.001)
+					(thickness 0.15)
 				)
 			)
@@
 				(font
 					(size 0.001 0.001)
+					(thickness 0.15)
 				)
 			)
@@
 				(font
 					(size 0.001 0.001)
+					(thickness 0.15)
 				)
 			)
@@
 				(font
 					(size 0.001 0.001)
+					(thickness 0.15)
 				)
 			)
@@
 				(font
 					(size 0.001 0.001)
+					(thickness 0.15)
 				)
 			)
@@
 				(font
 					(size 0.001 0.001)
+					(thickness 0.15)
 				)
 			)
@@
 				(font
 					(size 0.001 0.001)
+					(thickness 0.15)
 				)
 			)
@@
 				(font
 					(size 0.001 0.001)
+					(thickness 0.15)
 				)
 			)
@@
 	(footprint "Resistor_SMD:R_0402_1005Metric"
 		(layer "F.Cu")
-		(at 123.5 96.82 180)
+		(at 122.97 95.29 180)
 		(descr "Resistor SMD 0402 (1005 Metric), square (rectangular) end terminal, IPC-7351 nominal, (Body size source: IPC-SM-782 page 72, https://www.pcb-3d.com/wordpress/wp-content/uploads/ipc-sm-782a_amendment_1_and_2.pdf), generated with kicad-footprint-generator")
 		(tags "resistor")
@@
 				(font
 					(size 0.001 0.001)
+					(thickness 0.15)
 				)
 			)
@@
 				(font
 					(size 0.001 0.001)
+					(thickness 0.15)
 				)
 			)
@@
 	)
 	(segment
-		(start 118.8725 95.84)
+		(start 118.6225 96.09)
 		(end 118.12 96.5925)
 		(width 0.4)
@@
 	)
 	(segment
+		(start 118.6225 94.36)
+		(end 118.6225 96.09)
+		(width 0.4)
+		(layer "F.Cu")
+		(net 2)
+	)
+	(segment
 		(start 174.494 118.756)
 		(end 174.494 117.896)
@@
 	)
 	(via
-		(at 116.84 93.98)
-		(size 0.6)
-		(drill 0.3)
-		(layers "F.Cu" "B.Cu")
-		(free yes)
-		(net 3)
-	)
-	(via
 		(at 172.72 63.5)
 		(size 0.6)
@@
 	)
 	(segment
-		(start 122.96 96.79)
-		(end 122.99 96.82)
+		(start 120.5175 95.29)
+		(end 122.46 95.29)
 		(width 0.4)
 		(layer "F.Cu")
@@
 	)
 	(segment
-		(start 120.7475 96.79)
-		(end 122.96 96.79)
+		(start 120.4975 95.31)
+		(end 120.5175 95.29)
 		(width 0.4)
 		(layer "F.Cu")
@@
 	)
 	(segment
-		(start 134.22 92.66)
-		(end 132.8238 94.0562)
+		(start 132.8238 94.0562)
+		(end 124.3138 94.0562)
 		(width 0.4)
 		(layer "F.Cu")
@@
 	)
 	(segment
-		(start 132.8238 94.0562)
-		(end 124.3138 94.0562)
+		(start 134.22 75.06)
+		(end 134.22 92.66)
 		(width 0.4)
 		(layer "F.Cu")
@@
 	)
 	(segment
-		(start 134.22 75.06)
-		(end 134.22 92.66)
+		(start 134.22 92.66)
+		(end 132.8238 94.0562)
 		(width 0.4)
 		(layer "F.Cu")
@@
 	)
 	(segment
-		(start 124.3138 94.0562)
-		(end 124.01 94.36)
+		(start 124.01 94.36)
+		(end 124.01 94.76)
+		(width 0.4)
+		(layer "F.Cu")
+		(net 58)
+	)
+	(segment
+		(start 124.01 94.76)
+		(end 123.48 95.29)
 		(width 0.4)
 		(layer "F.Cu")
@@
 	)
 	(segment
-		(start 124.01 94.36)
-		(end 124.01 96.82)
+		(start 124.3138 94.0562)
+		(end 124.01 94.36)
 		(width 0.4)
 		(layer "F.Cu")

Commit message: some updates
Parts:
- removed BZ1: Buzzer, Buzzer_Beeper:Buzzer_12x9.5RM7.6
- removed the G*** at (121.9, 112.2)
- removed Q1: SS8050, Package_TO_SOT_SMD:SOT-23
- removed kibuzzard-696A19CC: G***, kibuzzard-696A19CC
- removed kibuzzard-696A1A13: G***, kibuzzard-696A1A13
- added C6: 100nF, Capacitor_SMD:C_0402_1005Metric, F.Cu at (123.1, 99.3)
- added CN10: IO, Connector_PinSocket_2.54mm:PinSocket_1x07_P2.54mm_Vertical, F.Cu at (153.7, 57.1)
- added CN11: QWIIC, Connector_JST:JST_SH_SM04B-SRSS-TB_1x04-1MP_P1.00mm_Horizontal, F.Cu at (117.8, 111.3)
- added G***: LOGO, logo:cyber, F.Cu at (127.6, 102.7)
- added G***: LOGO, logo:qwiic, F.Cu at (122.6, 111.1)
- added LD15: Led Blue, LED_SMD:LED_0603_1608Metric, F.Cu at (120.4, 85.7)
- added LD16: Led Blue, LED_SMD:LED_0603_1608Metric, F.Cu at (120.4, 88.6)
- added R32: 1k, Resistor_SMD:R_0402_1005Metric, F.Cu at (117.2, 88.6)
- added U7: ATECC608A-SSHDA, Package_SO:SOIC-8_3.9x4.9mm_P1.27mm, F.Cu at (121.3, 102.9)
- added kibuzzard-69594DEB: G***, kibuzzard-69594DEB, F.Cu at (187.8, 78.7)
- added kibuzzard-69594DEB: G***, kibuzzard-69594DEB, F.Cu at (116.6, 103.1)
- added kibuzzard-69594DEB: G***, kibuzzard-69594DEB, F.Cu at (187.8, 96.5)
- added kibuzzard-69908B33: G***, kibuzzard-69908B33, F.Cu at (194.2, 49.6)
- added kibuzzard-69908F16: G***, kibuzzard-69908F16, F.Cu at (125.9, 87.1)
- added kibuzzard-69908F24: G***, kibuzzard-69908F24, F.Cu at (123.4, 85.7)
- added kibuzzard-69908F2A: G***, kibuzzard-69908F2A, F.Cu at (123.5, 88.6)
- added kibuzzard-69909054: G***, kibuzzard-69909054, F.Cu at (119.7, 99.2)
- added kibuzzard-69909E2E: G***, kibuzzard-69909E2E, F.Cu at (156.2, 49.5)
- LD1, LD2, LD3, LD4, LD5, LD6: value O1_G -> Led Blue
- LD10, LD12, LD14: value Tx -> Led Blue
- LD11, LD13, LD9: value Rx -> Led Blue
- LD7: value 3v3 -> Led Red
- LD8: value 5v -> Led Red
- moved kibuzzard-69594DEB 27.2 mm to (184.0, 39.6), turned to 0 degrees
- moved R17 11.2 mm to (117.2, 85.7)
- moved R22 7.48 mm to (118.2, 97.0)
- moved SW4 7.48 mm to (119.8, 94.4)
- moved kibuzzard-69594C94 7.30 mm to (123.7, 94.3)
- moved G*** 0.61 mm to (165.1, 94.8)
Connections:
- D2 pad 2: /Lin_Vbat -> /Lin_Vcc
- JP4 pad 2: Net-(JP4-C) -> /Lin_Vcc
- MODULE1 pad 22: unconnected-(MODULE1-PC13-Pad22) -> Net-(CN10-Pin_2)
- MODULE1 pad 23: unconnected-(MODULE1-PC14-Pad23) -> Net-(CN10-Pin_3)
- MODULE1 pad 24: unconnected-(MODULE1-PC15-Pad24) -> Net-(CN10-Pin_4)
- R17 pad 1: /PA15 -> Net-(LD15-K)
- R17 pad 2: Net-(Q1-B) -> /CANRX
- U5 pad 7: Net-(JP4-C) -> /Lin_Vcc
Routing:
- net /5V: track 120.7 -> 193.2 mm, vias 6 -> 7
- net /SCL1: track 163.4 -> 210.7 mm, vias 3 -> 5
- net Net-(CN10-Pin_2): track 0.00 -> 44.6 mm, vias 0 -> 1
- net Net-(CN10-Pin_3): track 0.00 -> 43.8 mm, vias 0 -> 1
- net /SDA1: track 151.2 -> 193.3 mm
- net Net-(CN10-Pin_4): track 0.00 -> 41.5 mm
- net /3V3: track 330.4 -> 358.9 mm, vias 14 -> 15
- net /CANTX: track 26.6 -> 44.6 mm, vias 1 -> 2
- net /CANRX: track 26.8 -> 44.7 mm, vias 1 -> 2
- net /PA15: track 42.3 -> 25.1 mm, vias 2 -> 0
- net /Lin_Vcc: track 0.00 -> 17.0 mm, vias 0 -> 1
- net Net-(JP4-C): track 15.9 -> 0.00 mm, vias 1 -> 0
- net Net-(BZ1--): track 9.99 -> 0.00 mm
- net /Lin_Vbat: track 14.8 -> 9.16 mm
- net /WKUP: track 35.7 -> 39.4 mm
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